File: rasle.sch (KiCad schematic (older format))
At the start: 69 parts, among them J1 Power, J10 BUTTON4, J11 BUTTON_PWR, J12 External relay, J14 Conn_01x02_Male, J15 Conn_01x02_Male, J2 FAN, J3 LED1, J4 WS2812, J5 LED2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

Commit message: Added manufacturing files
Parts:
- added J13: Reset disable, Pin_Headers:Pin_Header_Straight_1x02, symbol Connector:Conn_01x02_Male
- MK1, MK2, MK3, MK4: symbol Mechanical:Mounting_Hole -> Mechanical:MountingHole
Connections:
- net labels added: RESET
- wire segments 165 -> 167
Changed lines of the file:
@@
 EESchema Schematic File Version 4
-LIBS:gamehat2-cache
 EELAYER 26 0
 EELAYER END
@@
 ID_SD and ID_SC PINS:\nThese pins are reserved for HAT ID EEPROM.\n\nAt boot time this I2C interface will be\ninterrogated to look for an EEPROM\nthat identifes the attached board and\nallows automagic setup of the GPIOs\n(and optionally, Linux drivers).\n\nDO NOT USE these pins for anything other\nthan attaching an I2C ID EEPROM. Leave\nunconnected if ID EEPROM not required.
 $Comp
-L Mechanical:Mounting_Hole MK1
+L Mechanical:MountingHole MK1
 U 1 1 5834FB2E
 P 3000 7200
@@
 $EndComp
 $Comp
-L Mechanical:Mounting_Hole MK3
+L Mechanical:MountingHole MK3
 U 1 1 5834FBEF
 P 3450 7200
@@
 $EndComp
 $Comp
-L Mechanical:Mounting_Hole MK2
+L Mechanical:MountingHole MK2
 U 1 1 5834FC19
 P 3000 7400
@@
 $EndComp
 $Comp
-L Mechanical:Mounting_Hole MK4
+L Mechanical:MountingHole MK4
 U 1 1 5834FC4F
 P 3450 7400
@@
 L Connector:Conn_01x03_Male J12
 U 1 1 5BA56664
-P 3800 6200
-F 0 "J12" H 3906 6478 50  0000 C CNN
-F 1 "External relay" V 3700 6250 50  0000 C CNN
-F 2 "Connectors_JST_PH:Connectors_JST_B3B-PH-K" H 3800 6200 50  0001 C CNN
-F 3 "~" H 3800 6200 50  0001 C CNN
-	1    3800 6200
+P 3800 6100
+F 0 "J12" H 3906 6378 50  0000 C CNN
+F 1 "External relay" V 3700 6150 50  0000 C CNN
+F 2 "Connectors_JST_PH:Connectors_JST_B3B-PH-K" H 3800 6100 50  0001 C CNN
+F 3 "~" H 3800 6100 50  0001 C CNN
+	1    3800 6100
 	1    0    0    -1
 $EndComp
 Text Label 6700 3700 0    50   ~ 0
 POWER
-Text Label 4000 6200 0    50   ~ 0
+Text Label 4000 6100 0    50   ~ 0
 POWER
 $Comp
 L power:+5V #PWR0115
 U 1 1 5BA56ACA
-P 4000 6000
-F 0 "#PWR0115" H 4000 5850 50  0001 C CNN
-F 1 "+5V" H 4015 6173 50  0000 C CNN
-F 2 "" H 4000 6000 50  0001 C CNN
-F 3 "" H 4000 6000 50  0001 C CNN
-	1    4000 6000
+P 4000 5900
+F 0 "#PWR0115" H 4000 5750 50  0001 C CNN
+F 1 "+5V" H 4015 6073 50  0000 C CNN
+F 2 "" H 4000 5900 50  0001 C CNN
+F 3 "" H 4000 5900 50  0001 C CNN
+	1    4000 5900
 	1    0    0    -1
 $EndComp
@@
 L power:GND #PWR0116
 U 1 1 5BA56B88
-P 4000 6400
-F 0 "#PWR0116" H 4000 6150 50  0001 C CNN
-F 1 "GND" H 4005 6227 50  0000 C CNN
-F 2 "" H 4000 6400 50  0001 C CNN
-F 3 "" H 4000 6400 50  0001 C CNN
-	1    4000 6400
-	1    0    0    -1
-$EndComp
-Wire Wire Line
-	4000 6400 4000 6300
+P 4000 6300
+F 0 "#PWR0116" H 4000 6050 50  0001 C CNN
+F 1 "GND" H 4005 6127 50  0000 C CNN
+F 2 "" H 4000 6300 50  0001 C CNN
+F 3 "" H 4000 6300 50  0001 C CNN
+	1    4000 6300
+	1    0    0    -1
+$EndComp
+Wire Wire Line
+	4000 6300 4000 6200
 Wire Wire Line
 	6100 2400 6100 2300
@@
 FAN
 Wire Wire Line
-	4000 6100 4000 6000
+	4000 6000 4000 5900
 $Comp
 L power:GND #PWR0129
@@
 U 1 1 5BAAE61A
 P 7600 3500
-F 0 "C15" V 7348 3500 50  0000 C CNN
-F 1 "C" V 7439 3500 50  0000 C CNN
+F 0 "C15" V 7750 3500 50  0000 C CNN
+F 1 "C" V 7850 3500 50  0000 C CNN
 F 2 "Capacitors_SMD:C_0805" H 7638 3350 50  0001 C CNN
 F 3 "~" H 7600 3500 50  0001 C CNN
@@
 Text Label 6700 2800 0    50   ~ 0
 FAN
-Text Label 1250 1400 2    50   ~ 0
-RESET_ATMEGA
 $Comp
 L power:GND #PWR0144
@@
 Wire Notes Line
 	8350 5850 8350 1950
+Text Label 1250 1400 2    50   ~ 0
+RESET
+$Comp
+L Connector:Conn_01x02_Male J13
+U 1 1 5BB825E5
+P 5050 1000
+F 0 "J13" H 5023 880 50  0000 R CNN
+F 1 "Reset disable" H 5023 971 50  0000 R CNN
+F 2 "Pin_Headers:Pin_Header_Straight_1x02" H 5050 1000 50  0001 C CNN
+F 3 "~" H 5050 1000 50  0001 C CNN
+	1    5050 1000
+	-1   0    0    1
+$EndComp
+Wire Wire Line
+	4850 1000 4850 1300
+Wire Wire Line
+	4850 650  4850 900
+Text Label 4850 650  0    50   ~ 0
+RESET
 $EndSCHEMATC

Commit message: Added EEPROM for HAT compatability
Parts:
- removed C13: C, Capacitors_SMD:C_0805, symbol Device:C
- added R16, R17: R, Resistors_SMD:R_0603, symbol Device:R
- added U5: 24AA02-OT, TO_SOT_Packages_SMD:SOT-23-5, symbol Memory_EEPROM:24AA02-OT
- C10, C11, C12, C14, C15, C3, C4, C5, C6, C7, C8, C9: footprint Capacitors_SMD:C_0805 -> Capacitors_SMD:C_0603
- R1, R10, R11, R12, R13, R14, R15, R18, R2, R21, R3, R4, R5, R6, R7, R8, R9: footprint Resistors_SMD:R_0805 -> Resistors_SMD:R_0603
Connections:
- wire segments 167 -> 170

Commit message: Added RTC chip for timekeeping
Parts:
- added J16: Conn_01x02_Male, Resistors_SMD:R_1206_HandSoldering, symbol Connector:Conn_01x02_Male
- added U6: DS3231M, Housings_SOIC:SOIC-16_7.5x10.3mm_Pitch1.27mm, symbol Timer_RTC:DS3231M
Connections:
- net labels added: +BATT, SCL, SDA
- wire segments 170 -> 171
- no-connect marks 0 -> 1
Changed lines of the file:
@@
 Wire Wire Line
 	4800 5000 4650 5000
+$Comp
+L Timer_RTC:DS3231M U6
+U 1 1 5BB9D1EF
+P 4550 7150
+F 0 "U6" H 4550 6664 50  0000 C CNN
+F 1 "DS3231M" H 4550 6573 50  0000 C CNN
+F 2 "Housings_SOIC:SOIC-16_7.5x10.3mm_Pitch1.27mm" H 4550 6550 50  0001 C CNN
+F 3 "http://datasheets.maximintegrated.com/en/ds/DS3231.pdf" H 4820 7200 50  0001 C CNN
+	1    4550 7150
+	1    0    0    -1
+$EndComp
+Text Label 1250 1200 2    50   ~ 0
+SDA
+Text Label 1250 1300 2    50   ~ 0
+SCL
+Text Label 4050 6950 2    50   ~ 0
+SCL
+Text Label 4050 7050 2    50   ~ 0
+SDA
+$Comp
+L gamehat2:+3V3 #PWR0160
+U 1 1 5BB9E001
+P 4450 6750
+F 0 "#PWR0160" H 4450 6600 50  0001 C CNN
+F 1 "+3V3" H 4465 6923 50  0000 C CNN
+F 2 "" H 4450 6750 50  0000 C CNN
+F 3 "" H 4450 6750 50  0000 C CNN
+	1    4450 6750
+	1    0    0    -1
+$EndComp
+$Comp
+L gamehat2:GND #PWR0161
+U 1 1 5BB9E128
+P 4550 7550
+F 0 "#PWR0161" H 4550 7300 50  0001 C CNN
+F 1 "GND" H 4555 7377 50  0000 C CNN
+F 2 "" H 4550 7550 50  0000 C CNN
+F 3 "" H 4550 7550 50  0000 C CNN
+	1    4550 7550
+	1    0    0    -1
+$EndComp
+NoConn ~ 4500 5800
+$Comp
+L power:+BATT #PWR0162
+U 1 1 5BBC1E9D
+P 4550 6450
+F 0 "#PWR0162" H 4550 6300 50  0001 C CNN
+F 1 "+BATT" H 4565 6623 50  0000 C CNN
+F 2 "" H 4550 6450 50  0001 C CNN
+F 3 "" H 4550 6450 50  0001 C CNN
+	1    4550 6450
+	1    0    0    -1
+$EndComp
+Wire Wire Line
+	4550 6450 4550 6750
+$Comp
+L Connector:Conn_01x02_Male J16
+U 1 1 5BBC98A4
+P 5450 7500
+F 0 "J16" H 5423 7380 50  0000 R CNN
+F 1 "Conn_01x02_Male" H 5423 7471 50  0000 R CNN
+F 2 "Resistors_SMD:R_1206_HandSoldering" H 5450 7500 50  0001 C CNN
+F 3 "~" H 5450 7500 50  0001 C CNN
+	1    5450 7500
+	-1   0    0    1
+$EndComp
+$Comp
+L gamehat2:GND #PWR0163
+U 1 1 5BBC9A7E
+P 5250 7500
+F 0 "#PWR0163" H 5250 7250 50  0001 C CNN
+F 1 "GND" H 5255 7327 50  0000 C CNN
+F 2 "" H 5250 7500 50  0000 C CNN
+F 3 "" H 5250 7500 50  0000 C CNN
+	1    5250 7500
+	1    0    0    -1
+$EndComp
+$Comp
+L power:+BATT #PWR0164
+U 1 1 5BBC9B85
+P 5250 7400
+F 0 "#PWR0164" H 5250 7250 50  0001 C CNN
+F 1 "+BATT" H 5265 7573 50  0000 C CNN
+F 2 "" H 5250 7400 50  0001 C CNN
+F 3 "" H 5250 7400 50  0001 C CNN
+	1    5250 7400
+	1    0    0    -1
+$EndComp
 $EndSCHEMATC

Commit message: Removed RTC chip as it is not necessary
Parts:
- removed J16: Conn_01x02_Male, Resistors_SMD:R_1206_HandSoldering, symbol Connector:Conn_01x02_Male
- removed U6: DS3231M, Housings_SOIC:SOIC-16_7.5x10.3mm_Pitch1.27mm, symbol Timer_RTC:DS3231M
- added D1: LED, LEDs:LED-0603, symbol Device:LED
- added R19: 220R, Resistors_SMD:R_0603, symbol Device:R
- C1, C2: value CP -> 10uF
- C10, C11, C12, C3, C4, C5, C6, C7, C8, C9: value C -> 100nF
- C14, C15: value C -> 22pF
- C16, C17, C18, C19: value C -> 220nF
- J2: footprint adafruit:FAN -> Connectors_JST_PH:Connectors_JST_B2B-PH-K
- J4: footprint Connectors_JST_PH:Connectors_JST_B3B-PH-K -> Pin_Headers:Pin_Header_Straight_1x03
- LED1: renamed from J3; value LED1 -> PWM; footprint Connectors_JST_PH:Connectors_JST_B2B-PH-K -> Pin_Headers:Pin_Header_Straight_1x02
- LED2: renamed from J5; value LED2 -> PWM; footprint Connectors_JST_PH:Connectors_JST_B2B-PH-K -> Pin_Headers:Pin_Header_Straight_1x02
- LED3: renamed from J6; value LED3 -> PWM; footprint Connectors_JST_PH:Connectors_JST_B2B-PH-K -> Pin_Headers:Pin_Header_Straight_1x02
- Q1, Q2, Q3, Q4: Manufacturer (none) -> Diodes Inc; Manufacturer no (none) -> DMN2041L-7; Mouser No (none) -> '621-DMN2041L-7
- R1, R2, R3, R7: value R -> 0R
- R11, R12, R13, R14, R15, R18, R4, R5, R6, R8: value R -> 10k
- R16, R17: value R -> 4k7
- Y1: footprint Crystals:Crystal_HC49-SD_SMD -> mysensors_obscurities:XTAL_3.2x1.5mm
Connections:
- net labels removed: +BATT
- wire segments 171 -> 169

Commit message: Connected atmega to all buttons, so it can listen to the same button events as RPI
Changed lines of the file:
@@
 	1    0    0    -1
 $EndComp
-Text Label 6700 3700 0    50   ~ 0
+Text Label 6700 4600 0    50   ~ 0
 POWER
 Text Label 4000 6100 0    50   ~ 0
@@
 Text Label 3950 1600 0    50   ~ 0
 BCLK
-Text Label 6700 3800 0    50   ~ 0
-GPIO23(GEN4)
-Text Label 6700 3900 0    50   ~ 0
-GPIO24(GEN5)
 Text Label 4850 1300 0    50   ~ 0
 RESET_ATMEGA
@@
 	1    0    0    -1
 $EndComp
+Text Label 6700 3900 0    50   ~ 0
+BUTTON4
+Text Label 6700 3800 0    50   ~ 0
+BUTTON2
+Text Label 6700 3700 0    50   ~ 0
+BUTTON3
+Text Label 6700 2900 0    50   ~ 0
+BUTTON1
 $EndSCHEMATC
